Commit message: Add real-hardware arm bringup

File: ra_ws/src/so_arm_moveit_config/config/so101_new_calib.ros2_control.xacro (robot description, xacro)
@@ -1,14 +1,31 @@
 <?xml version="1.0"?>
 <robot xmlns:xacro="http://www.ros.org/wiki/xacro">
-    <xacro:macro name="so101_new_calib_ros2_control" params="name initial_positions_file">
+    <!--
+      ros2_control_hardware_type selects the hardware interface:
+        "isaac"   -> topic_based bridge to Isaac Sim (simulation, DEFAULT)
+        "feetech" -> real STS3215 servos over the serial bus (physical arm)
+      Sim behaviour is unchanged when the arg is left at its default.
+    -->
+    <xacro:macro name="so101_new_calib_ros2_control" params="name initial_positions_file ros2_control_hardware_type:=isaac">
         <xacro:property name="initial_positions" value="${xacro.load_yaml(initial_positions_file)['initial_positions']}"/>
         <ros2_control name="${name}" type="system">
             <hardware>
-                <!-- By default, set up controllers for simulation. This won't work on real hardware -->
-                <plugin>topic_based_ros2_control/TopicBasedSystem</plugin>
-                <param name="joint_commands_topic">/isaac_joint_commands</param>
-                <param name="joint_states_topic">/isaac_joint_states</param>
+                <xacro:if value="${ros2_control_hardware_type == 'isaac'}">
+                    <!-- Simulation: bridge to Isaac Sim. This won't work on real hardware. -->
+                    <plugin>topic_based_ros2_control/TopicBasedSystem</plugin>
+                    <param name="joint_commands_topic">/isaac_joint_commands</param>
+                    <param name="joint_states_topic">/isaac_joint_states</param>
+                </xacro:if>
+                <xacro:if value="${ros2_control_hardware_type == 'feetech'}">
+                    <!-- Real arm: Feetech STS3215 servos on the serial bus.
+                         Per-robot calibration (homing_offset / range_min / range_max)
+                         lives in follower_joints.yaml, matched to each joint by servo id. -->
+                    <plugin>feetech_ros2_driver/FeetechHardwareInterface</plugin>
+                    <param name="usb_port">/dev/ttyACM0</param>
+                    <param name="joint_config_file">$(find so_arm_moveit_config)/config/follower_joints.yaml</param>
+                </xacro:if>
             </hardware>
             <joint name="Rotation">
+                <xacro:if value="${ros2_control_hardware_type == 'feetech'}"><param name="id">1</param></xacro:if>
                 <command_interface name="position"/>
                 <state_interface name="position">
@@ -18,4 +35,5 @@
             </joint>
             <joint name="Pitch">
+                <xacro:if value="${ros2_control_hardware_type == 'feetech'}"><param name="id">2</param></xacro:if>
                 <command_interface name="position"/>
                 <state_interface name="position">
@@ -25,4 +43,5 @@
             </joint>
             <joint name="Elbow">
+                <xacro:if value="${ros2_control_hardware_type == 'feetech'}"><param name="id">3</param></xacro:if>
                 <command_interface name="position"/>
                 <state_interface name="position">
@@ -32,4 +51,5 @@
             </joint>
             <joint name="Wrist_Pitch">
+                <xacro:if value="${ros2_control_hardware_type == 'feetech'}"><param name="id">4</param></xacro:if>
                 <command_interface name="position"/>
                 <state_interface name="position">
@@ -39,4 +59,5 @@
             </joint>
             <joint name="Wrist_Roll">
+                <xacro:if value="${ros2_control_hardware_type == 'feetech'}"><param name="id">5</param></xacro:if>
                 <command_interface name="position"/>
                 <state_interface name="position">
@@ -46,4 +67,5 @@
             </joint>
             <joint name="Jaw">
+                <xacro:if value="${ros2_control_hardware_type == 'feetech'}"><param name="id">6</param></xacro:if>
                 <command_interface name="position"/>
                 <state_interface name="position">

File: ra_ws/src/so_arm_moveit_config/config/so101_new_calib.urdf.xacro (robot description, xacro)
@@ -2,8 +2,10 @@
 <robot xmlns:xacro="http://www.ros.org/wiki/xacro" name="so101_new_calib">
     <xacro:arg name="initial_positions_file" default="initial_positions.yaml" />
+    <!-- "isaac" = Isaac Sim bridge (default), "feetech" = real STS3215 hardware -->
+    <xacro:arg name="ros2_control_hardware_type" default="isaac" />
     <!-- Import so101_new_calib urdf file -->
     <xacro:include filename="$(find so_arm_description)/urdf/so101_new_calib.urdf" />
     <!-- Import control_xacro -->
     <xacro:include filename="so101_new_calib.ros2_control.xacro" />
-    <xacro:so101_new_calib_ros2_control name="FakeSystem" initial_positions_file="$(arg initial_positions_file)"/>
+    <xacro:so101_new_calib_ros2_control name="FakeSystem" initial_positions_file="$(arg initial_positions_file)" ros2_control_hardware_type="$(arg ros2_control_hardware_type)"/>
 </robot>
